File: Rev 1.sch (EAGLE design)
At the start: 63 parts, among them P5 EJECTION_CHARGE, P6 EJECTION_CHARGE, P7 EJECTION_CHARGE, P8 EJECTION_CHARGE, Q1 MMBT3904, Q2 BCV27, Q3 MMBT3904, Q4 BCV27, Q5 MMBT3904, Q6 MMBT3904, Q7 MMBT3906, Q8 MMBT3904, U1 LFXP6E-3FN256C, U2 LPS22HH, U3 LSM6DS3, U4 MS5637-02BA03, U5 JF2, U6 RFM69HCW, Y1 DSC1122B

Commit message: Finished up schematic
Parts:
- added AE5: ANTENNA, Bulkhead Flight Computer:ANTENNA
- added AE6: 5-1814832-1, Bulkhead Flight Computer:5-1814832-1
- added BT1, BT2: 18650, Bulkhead Flight Computer:18650
- added C19, C32, C33, C34, C35, C36, C37, C38, C39, C40, C46, C50, C63, C64, C65: 0.1uF, Bulkhead Flight Computer:CAPACITOR0805
- added C20, C21: 22pF, Bulkhead Flight Computer:CAPACITOR0805
- added C22, C23, C24, C25, C26, C27, C28, C29, C30, C31, C61, C62: 10nF, Bulkhead Flight Computer:CAPACITOR0805
- added C41, C44, C45, C51, C52, C53, C54, C59, C67: 1uF, Bulkhead Flight Computer:CAPACITOR0805
- added C42, C43: 1F, Bulkhead Flight Computer:ELECTROLYTIC
- added C47, C48, C49: 2.2uF, Bulkhead Flight Computer:CAPACITOR0805
- added C55: 4.7uF, Bulkhead Flight Computer:CAPACITOR0805
- added C56, C66, C70: 10uF, Bulkhead Flight Computer:CAPACITOR0805
- added C57: 8.2pF, Bulkhead Flight Computer:CAPACITOR0805
- added C58, C68: 6.2pF, Bulkhead Flight Computer:CAPACITOR0805
- added C60: 100pF, Bulkhead Flight Computer:CAPACITOR0805
- added C69: 22uF, Bulkhead Flight Computer:CAPACITOR0805
- added D3, D4, D5, D6: LED, Bulkhead Flight Computer:LED
- added FL1: SAWAFS915.0W03-TS4, Bulkhead Flight Computer:SAWAFS915.0W03-TS4
- added J1: USB, Bulkhead Flight Computer:USB
- added JP3, JP5: (no value), Bulkhead Flight Computer:PINHD-1X4
- added JP4: (no value), Bulkhead Flight Computer:PINHD-1X7
- added JP6: (no value), Bulkhead Flight Computer:PINHD-1X2
- added JP7, JP8: (no value), Bulkhead Flight Computer:PINHD-1X3
- added L2: 2.7nH, Bulkhead Flight Computer:INDUCTOR
- added L3: 33nH, Bulkhead Flight Computer:INDUCTOR
- added L4: 5.6nH, Bulkhead Flight Computer:INDUCTOR
- added L5, L6: 840nH, Bulkhead Flight Computer:INDUCTOR
- added L7: 0.47uH, Bulkhead Flight Computer:INDUCTOR
- added P1: SDCARD, Bulkhead Flight Computer:SDCARD
- added Q10, Q11, Q12, Q13, Q15, Q16, Q17, Q18: MMBT3904, Bulkhead Flight Computer:MMBT3904
- added Q14: PHOTOTRANSISTOR, Bulkhead Flight Computer:PHOTOTRANSISTOR
- added Q19: P-MOSFETTPH1R712MD, Bulkhead Flight Computer:P-MOSFETTPH1R712MD
- added Q20: TAV-541+, Bulkhead Flight Computer:TAV-541+
- added Q9: BCV27, Bulkhead Flight Computer:BCV27
- added R17: 10R, Bulkhead Flight Computer:RESISTOR0805
- added R18, R19, R39, R43, R44, R45, R46, R53: 10k, Bulkhead Flight Computer:RESISTOR0805
- added R20, R21, R22, R23, R24, R25, R26, R27, R28, R29, R30: 4.7k, Bulkhead Flight Computer:RESISTOR0805
- added R31, R32, R33, R34, R54: (no value), Bulkhead Flight Computer:RESISTOR0805
- added R35: 330k, Bulkhead Flight Computer:RESISTOR0805
- added R36, R38, R55, R57: 100k, Bulkhead Flight Computer:RESISTOR0805
- added R37: 33R, Bulkhead Flight Computer:RESISTOR0805
- added R40, R49: 13k, Bulkhead Flight Computer:RESISTOR0805
- added R41: 15k, Bulkhead Flight Computer:RESISTOR0805
- added R42, R47, R50: 0R, Bulkhead Flight Computer:RESISTOR0805
- added R48: 18k, Bulkhead Flight Computer:RESISTOR0805
- added R51: 1.5k, Bulkhead Flight Computer:RESISTOR0805
- added R52: 12k, Bulkhead Flight Computer:RESISTOR0805
- added R56: 200k, Bulkhead Flight Computer:RESISTOR0805
- added TP1, TP2: TOUCH_POINTBTN, Bulkhead Flight Computer:TOUCH_POINTBTN
- added TP10, TP11, TP3, TP4, TP5, TP6, TP7, TP8, TP9: TOUCH_POINTSTRIP, Bulkhead Flight Computer:TOUCH_POINTSTRIP
- added U10: LTV-357T, Bulkhead Flight Computer:LTV-357T
- added U11: LDO_ADJLM317BD2TR4G, Bulkhead Flight Computer:LDO_ADJLM317BD2TR4G
- added U12: LDO_ENLDLN025PU18R, Bulkhead Flight Computer:LDO_ENLDLN025PU18R
- added U13: LTC2361, Bulkhead Flight Computer:LTC2361
- added U14: LDOAP2125, Bulkhead Flight Computer:LDOAP2125
- added U15: LDO_ENAP7365, Bulkhead Flight Computer:LDO_ENAP7365
- added U16: AP3417C, Bulkhead Flight Computer:AP3417C
- added U17: GVA-91+, Bulkhead Flight Computer:GVA-91+
- added U18: MIC47050, Bulkhead Flight Computer:MIC47050
- added U19: FAN48610, Bulkhead Flight Computer:FAN48610
- added U7: ATMEGA328PB32-TQFP, Bulkhead Flight Computer:ATMEGA328PB32-TQFP
- added U8: AT42QT1110, Bulkhead Flight Computer:AT42QT1110
- added U9: RFM69HCW, Bulkhead Flight Computer:RFM69HCW
- added XTAL1: CRYSTAL, Bulkhead Flight Computer:CRYSTAL
- C13: value 27pF -> 10nF
- JP2: device Bulkhead Flight Computer:PINHD-1X2 -> Bulkhead Flight Computer:PINHD-1X4
- L1: value 35.5nH -> 2.2uH
- U2: value LPS22HH -> RPI-ZERO; device Bulkhead Flight Computer:LPS22HH -> Bulkhead Flight Computer:RPI-ZERO
Connections:
- net RF_CS renamed RF_RX_CS
- net RF_IO0 renamed RF_RX_IO0
- net RF_IO1 renamed RF_RX_IO1
- net RF_IO2 renamed RF_RX_IO2
- net RF_IO3 renamed RF_RX_IO3
- net RF_IO4 renamed RF_RX_IO4
- net RF_IO5 renamed RF_RX_IO5
- net RF_MISO renamed RF_RX_MISO
- net RF_MOSI renamed RF_RX_MOSI
- net RF_RST renamed RF_RX_RST
- net RF_SCK renamed RF_RX_SCK
- net SPEAKER renamed BUZZER
- removed net BARO_CS: U2.CS
- removed net BARO_DRDY: U2.DRDY
- removed net BARO_MISO: U2.SA0
- removed net BARO_MOSI: U2.SDA
- removed net BARO_SCLK: U2.SCL
- removed net CHARGE_OTHER_SIDE: JP2.2, P8.P$1
- removed net POWER_EN: R15.P$1
- new net +5V: C59.P$2, C60.P$2, C69.P$2, L3.P$2, U19.VOUT
- new net ADC_CONV: U13.CONV
- new net ADC_SCK: U13.SCK
- new net ADC_SDO: U13.SDO
- new net LED_ARM: Q13.B
- new net LED_G: Q11.B
- new net LED_LOCK: Q12.B
- new net LED_R: Q10.B
- new net MISO: JP4.2, U7.PB4, U8.MISO
- new net MOSI: JP4.1, U7.PB3, U8.MOSI
- new net N$18: AE5.P$1, Q9.E
- new net N$19: R19.P$1, U8.RESET
- new net N$20: Q9.C, R17.P$1
- new net N$21: C13.P$1, U8.SNS5
- new net N$22: C13.P$2, R20.P$1, U8.SNS5K
- new net N$23: C27.P$2, R26.P$1, U8.SNS6K
- new net N$24: C28.P$2, R27.P$1, U8.SNS7K
- new net N$25: C29.P$2, R28.P$1, U8.SNS8K
- new net N$26: C30.P$2, R29.P$1, U8.SNS9K
- new net N$27: C31.P$2, R30.P$1, U8.SNS10K
- new net N$28: C22.P$2, R21.P$1, U8.SNS4K
- new net N$29: C23.P$2, R22.P$1, U8.SNS3K
- new net N$30: C24.P$2, R23.P$1, U8.SNS2K
- new net N$31: C25.P$2, R24.P$1, U8.SNS1K
- new net N$32: C26.P$2, R25.P$1, U8.SNS0K
- new net N$33: C27.P$1, U8.SNS6
- new net N$34: C28.P$1, U8.SNS7
- new net N$35: C29.P$1, U8.SNS8
- new net N$36: C30.P$1, U8.SNS9
- new net N$37: C31.P$1, U8.SNS10
- new net N$38: C22.P$1, U8.SNS4
- new net N$39: C23.P$1, U8.SNS3
- new net N$40: C24.P$1, U8.SNS2
- new net N$41: C25.P$1, U8.SNS1
- new net N$42: C26.P$1, U8.SNS0
- new net N$43: R30.P$2, TP11.1
- new net N$44: R29.P$2, TP10.1
- new net N$45: R28.P$2, TP9.1
- new net N$46: R27.P$2, TP8.1
- new net N$47: R26.P$2, TP7.1
- new net N$48: R20.P$2, TP6.1
- new net N$49: R21.P$2, TP5.1
- new net N$50: R22.P$2, TP4.1
- new net N$51: R23.P$2, TP3.1
- new net N$52: R24.P$2, TP2.1
- new net N$53: R25.P$2, TP1.1
- new net N$54: D3.OUT, Q10.C
- new net N$55: D3.IN, R31.P$1
- new net N$56: D4.OUT, Q11.C
- new net N$57: D4.IN, R32.P$1
- new net N$58: D5.OUT, Q12.C
- new net N$59: D5.IN, R33.P$1
- new net N$60: D6.OUT, Q13.C
- new net N$61: D6.IN, R34.P$1
- new net N$62: C57.P$2, L2.P$2, U9.ANT
- new net N$63: C33.P$2, U7.AREF
- new net N$64: JP5.3, P7.P$1
- new net N$65: JP5.4, P8.P$1
- new net N$66: Q14.E, Q15.B
- new net N$67: R37.P$1, U10.ANODE
- new net N$68: JP2.3, U10.COLLECTOR
- new net N$69: JP2.4, U10.EMITTER
- new net N$70: C14.P$2, C45.P$2, R12.P$2, R42.P$1, U12.OUT, U5.VDD
- new net N$71: Q16.C, U10.CATHODE
- new net N$72: D2.OUT, Q17.B
- new net N$73: R45.P$2, U15.EN
- new net N$74: R40.P$1, R41.P$2, U11.ADJ
- new net N$75: R43.P$2, U12.EN
- new net N$76: Q18.B, R15.P$1
- new net N$77: C41.P$2, C42.+, C43.+, C44.P$2, R40.P$2, R43.P$1, U11.OUT, U12.IN
- new net N$78: Q18.C, R47.P$1
- new net N$79: C62.P$2, L6.P$1, Q20.G
- new net N$80: R48.P$1, R49.P$2, U13.AIN
- new net N$81: C64.P$2, C67.P$2, L6.P$2, R51.P$2, U18.OUT
- new net N$82: C50.P$2, J1.+
- new net N$83: C50.P$1, J1.-
- new net N$84: R46.P$1, U16.EN
- new net N$85: C58.P$2, L3.P$1, U17.OUT
- new net N$86: L1.P$1, U16.LX
- new net N$87: R56.P$1, R57.P$2, U16.FB
- new net N$88: C61.P$2, U6.ANT
- new net N$89: AE4.OUT, C58.P$1, L4.P$2
- new net N$90: C61.P$1, L5.P$1, Q20.D
- new net N$91: R53.P$1, U18.EN
- new net N$92: R51.P$1, R52.P$2, U18.ADJ
- new net N$93: C62.P$1, FL1.OUT
- new net N$94: C68.P$2, FL1.IN
- new net N$95: AE6.OUT, C68.P$1
- new net N$96: L7.P$1, U19.SW
- new net N$97: R54.P$1, U19.EN
- new net ON: JP6.1, Q19.G, R47.P$2, R55.P$1
- new net OTHER_RX: JP2.2, R39.P$1
- new net OTHER_TX: Q16.B
- new net PHOTO: Q15.C, R38.P$1
- new net RESET: JP4.4, R18.P$1, U7.PC6
- new net RF_OUT: Q9.B
- new net RF_TX_CS: U9.NSS
- new net RF_TX_IO0: U9.DIO0
- new net RF_TX_IO1: U9.DIO1
- new net RF_TX_IO2: U9.DIO2
- new net RF_TX_IO3: U9.DIO3
- new net RF_TX_IO4: U9.DIO4
- new net RF_TX_IO5: U9.DIO5
- new net RF_TX_MISO: U9.MISO
- new net RF_TX_MOSI: U9.MOSI
- new net RF_TX_RST: U9.RESET
- new net RF_TX_SCK: U9.SCK
- new net RPI_RX: JP3.3, U2.RX
- new net RPI_TX: JP3.2, U2.TX
- new net RX: JP4.6, U7.PD0
- new net SCLK: JP4.3, U7.PB5, U8.SCK
- new net SD_CLK: P1.CLK
- new net SD_CMD: P1.CMD
- new net SD_DAT0: P1.DAT0
- new net SD_DAT1: P1.DAT1
- new net SD_DAT2: P1.DAT2
- new net SD_DAT3: P1.DAT3
- new net TOUCH_CS: U8.SS
- new net TOUCH_INT: U8.CHANGE
- new net TX: JP4.5, U7.PD1
- new net USB+: J1.D+
- new net USB-: J1.D-
- new net VBAT: BT2.+, C46.P$2, C55.P$2, C70.P$2, JP7.2, JP8.2, L7.P$2, Q19.S, R16.P$2, R50.P$1, R55.P$2, U16.VIN, U19.VIN
- new net VREF: R35.P$1, R36.P$2
- new net XTAL1: C20.P$2, U7.PB6, XTAL1.P$1
- new net XTAL2: C21.P$2, U7.PB7, XTAL1.P$2
- net +1V2: now also C54.P$2, C66.P$2, R53.P$2, U15.OUT, U18.IN
- net +1V8: now also C17.P$2, C37.P$2, C38.P$2, C39.P$2, C47.P$2, C48.P$2, C53.P$2, C56.P$2, C8.P$2, C9.P$2, L1.P$2, R37.P$2, R38.P$2, R39.P$2, R42.P$2, R44.P$2, R45.P$1, R56.P$2, U13.OVDD, U13.VREF, U15.IN, U3.VDD, U3.VDDIO, U4.VDD; no longer C14.P$2, R12.P$2, U5.VDD
- net +3V3: now also C32.P$2, C35.P$2, C49.P$2, C52.P$2, C63.P$2, C65.P$2, L5.P$2, P1.VDD, U13.VDD, U14.OUT, U18.BIAS, U9.3V3; no longer C5.P$2, C8.P$2, C9.P$2, U2.VDD, U2.VDDIO, U3.VDD, U3.VDDIO, U4.VDD
- net +3V7: now also BT1.+, C19.P$2, C34.P$2, C36.P$2, C40.P$2, C5.P$2, C51.P$2, JP3.1, JP5.1, Q14.C, Q19.D, R17.P$2, R18.P$2, R19.P$2, R31.P$2, R32.P$2, R33.P$2, R34.P$2, R35.P$2, R46.P$2, R48.P$2, R50.P$2, R54.P$2, U11.IN, U14.IN, U2.+5V, U7.AVCC, U7.VCC, U8.VDD; no longer C13.P$2, L1.P$2, P7.P$1, R16.P$2
- net CHARGE_SECONDARY: now also JP5.2; no longer JP2.1
- net GND: now also AE5.P$2, BT1.-, BT2.-, C19.P$1, C20.P$1, C21.P$1, C32.P$1, C33.P$1, C34.P$1, C35.P$1, C36.P$1, C37.P$1, C38.P$1, C39.P$1, C40.P$1, C41.P$1, C42.-, C43.-, C44.P$1, C45.P$1, C46.P$1, C47.P$1, C48.P$1, C49.P$1, C51.P$1, C52.P$1, C53.P$1, C54.P$1, C55.P$1, C56.P$1, C59.P$1, C60.P$1, C63.P$1, C64.P$1, C65.P$1, C66.P$1, C67.P$1, C69.P$1, C70.P$1, FL1.GND, JP2.1, JP3.4, JP4.7, JP6.2, JP7.1, JP7.3, JP8.1, JP8.3, L2.P$1, L4.P$1, P1.VSS, Q10.E, Q11.E, Q12.E, Q13.E, Q15.E, Q16.E, Q17.E, Q18.E, Q20.S, R36.P$1, R41.P$1, R49.P$1, R52.P$1, R57.P$1, U12.GND, U13.GND, U14.GND, U15.GND, U16.GND, U17.GND, U18.GND, U19.AGND, U19.PGND, U7.GND, U8.VSS, U9.GND; no longer AE4.GND, C13.P$1
- net N$17: now also C57.P$1, U17.IN; no longer AE4.OUT, U6.ANT
- net N$9: no longer L1.P$1
- net REMOTE_RF: now also Q17.C, R44.P$1; no longer C17.P$2, D2.OUT
Other:
- note added: "IO Pins to connect: 3.3V: RPI_TX RPI_RX SD_CMD SD_CLK SD_DAT0 SD_DAT1 SD_DAT2 SD_DAT3 FIRE_PRIMARY DETECT_PRIMARY FIRE_SECONDARY DETECT_SECONDARY RF_RX_MISO RF_RX_MOSI RF_RX_SCK RF_RX_CS RF_RX_RST RF_RX_IO0 RF_RX_IO1 RF_RX_IO2 RF_RX_IO3 RF_RX_IO4 RF_RX_IO5 RF_TX_MISO RF_TX_MOSI RF_TX_SCK RF_TX_CS RF_TX_RST RF_TX_IO0 RF_TX_IO1 RF_TX_IO2 RF_TX_IO3 RF_TX_IO4 RF_TX_IO5 BUZZER USB+ USB- OFF 1.8V: PHOT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"
- note added: "IO Pins to connect: RF_OUT LED_R LED_G LED_LOCK LED_ARM BUZZER TOUCH_CS TOUCH_INT (IRQ) VREF (ADC)"
- note added: "TODO: New IMU?"
